Commit message: limited joint ranges

File: ur5_demo_support/urdf/ur5_demo_robot.xacro (robot description, xacro)
@@ -8,5 +8,5 @@
   <xacro:property name="tool_tip_length" value="0.06"/>
   <xacro:property name="tool_extent_width" value="0.04"/>
-  <xacro:property name="tool_extent_length" value="0.07"/>
+  <xacro:property name="tool_extent_length" value="0.02"/>
   <xacro:property name="tool_body_width" value="0.04"/>
   <xacro:property name="tool_body_length" value="0.1"/>
@@ -15,5 +15,5 @@
   <xacro:include filename="$(find ur_description)/urdf/gazebo.urdf.xacro" />
   <!-- ur5 -->
-  <xacro:include filename="$(find ur_description)/urdf/ur5.urdf.xacro" />
+  <xacro:include filename="$(find ur5_demo_support)/urdf/ur5.urdf.xacro" />
   <!-- arm -->
   <xacro:ur5_robot prefix="" joint_limited="true"/>
@@ -53,15 +53,41 @@
       </material>
     </visual>
+    <collision>
+      <origin xyz="0 0 ${- tool_tip_length - 0.5*tool_body_length}" rpy="0 0 0"/>
+      <geometry>
+        <box size="${tool_body_width} ${tool_body_width} ${tool_body_length}"/>
+      </geometry>
+      <material name="yellow">
+        <color rgba="1 1 0 1"/>
+      </material>
+    </collision>
+    <collision>
+      <origin xyz="0 ${-0.5*tool_extent_length} ${-tool_tip_length - 0.5*tool_body_length}" rpy="${-0.5*PI} 0 0"/>
+      <geometry>
+        <cylinder radius="${0.5*tool_extent_width}" length="${tool_extent_length}"/>
+      </geometry>
+      <material name="yellow">
+        <color rgba="1 1 0 1"/>
+      </material>
+    </collision>
+    <collision>
+      <origin xyz="0 0 ${-0.5 * tool_tip_length}" rpy="0 0 0"/>
+      <geometry>
+        <cylinder radius="${tool_tip_width}" length="${tool_tip_length}"/>
+      </geometry>
+      <material name="yellow">
+        <color rgba="1 1 0 1"/>
+      </material>
+    </collision>
   </link>
-  <link name="flange_frame"/>
-  <joint name="wrist_to_flange" type="fixed">
-    <parent link="wrist_3_link"/>
-    <child link="flange_frame"/>
-    <origin xyz="0 ${flange_offset} 0" rpy="0 ${0.5*PI} 0"/>
-  </joint>
+  <!--<joint name="flange_to_tool" type="fixed">
+    <parent link="ee_link"/>
+    <child link="tool"/>
+    <origin xyz="${tool_length} 0 0 " rpy="0 ${0.5*PI} ${0}"/>
+  </joint>-->
   <joint name="flange_to_tool" type="fixed">
-    <parent link="flange_frame"/>
+    <parent link="ee_link"/>
     <child link="tool"/>
-    <origin xyz="${tool_length} ${tool_extent_length} 0" rpy="0 ${0.5*PI} 0"/>
+    <origin xyz="${tool_extent_length} 0 ${tool_length}" rpy="0 0 ${-0.5*PI}"/>
   </joint>
 </robot>

Commit message: modified the tool dimensions

File: ur5_demo_support/urdf/ur5_demo_robot.xacro (robot description, xacro)
@@ -6,9 +6,9 @@
   <xacro:property name="flange_offset" value="0.08"/>
   <xacro:property name="tool_tip_width" value="0.005"/>
-  <xacro:property name="tool_tip_length" value="0.06"/>
+  <xacro:property name="tool_tip_length" value="0.08"/>
   <xacro:property name="tool_extent_width" value="0.04"/>
   <xacro:property name="tool_extent_length" value="0.02"/>
   <xacro:property name="tool_body_width" value="0.04"/>
-  <xacro:property name="tool_body_length" value="0.1"/>
+  <xacro:property name="tool_body_length" value="0.06"/>
   <xacro:property name="tool_length" value="${0.5*tool_body_length + tool_tip_length}"/>
   <!-- common stuff -->
